File: schematics/schematic/schematic.kicad_sch (KiCad schematic)
At the start: 0 parts

Commit message: Commit WIP 1
Parts:
- added A1: Arduino_UNO_R3, Module:Arduino_UNO_R3, symbol MCU_Module:Arduino_UNO_R3
- added J1: USB_A, symbol Connector:USB_A
Connections:
- new net: A1.15 (D0/RX), J1.3 (D+)
- new net: A1.16 (D1/TX), J1.2 (D-)
- new net: A1.7 (GND), J1.4 (GND), J1.SH (Shield)
